File: P2/P2.brd (EAGLE design)
At the start: 68.6 x 53.3 mm, 12 parts

Commit message: Update P2.brd
Parts:
- added U2: (no value), AUTODESK_CIRCUITS_BREADBOARD:DIL16
Connections:
- removed net N$14 (its old number): PING2.2, R1.P$2, SERVO1.2, SERVO2.2, U1.5V
- removed net N$7 (its old number): D3.A, U1.12
- removed net N$8 (its old number): PING2.1, TILT1.2, U1.GND
- new net N$11: D3.A, U1.11
- new net N$13: PING2.1, TILT1.2, U1.GND, U2.4
- new net N$15: U1.2, U2.7
- new net N$16: U1.6, U2.1
- new net N$17: U1.8, U2.2
- new net N$18: U2.3
- new net N$19: U2.6
- net N$12: now also D2.A, U1.10; no longer U1.6
- net N$5: now also D1.A, U1.12; no longer D4.A, U1.11
- net N$6: now also D4.A, U1.13; no longer D1.A, U1.10
- net N$9: now also PING2.2, R1.P$2, SERVO1.2, SERVO2.2, U1.5V, U2.16, U2.8; no longer D2.A, U1.13
